File: LU Player Tracker Board V1/board.brd (EAGLE design)
At the start: 247 x 191.8 mm, 24 parts, among them IC2 TXU0304PWR, U3 ESP32-S3-WROOM-1-N16R2

Commit message: Added all the main lines
Parts:
- moved U3 8.06 mm to (-38.3, -12.1)
Other:
- board text removed: "not"

Commit message: update
Parts:
- removed VOLTAGE_REG: TLS850B0TBV33ATMA1, SamacSys_Parts:TLS850B0TBV33ATMA1
- added C5, C6: .1uF, adafruit:C0402
- added C7, C8: 1uF, adafruit:C0402
- added D1, D2: ESD9L5.0ST5G, SamacSys_Parts:SODFL1006X40N
- added DS1: HDSM-291C, SamacSys_Parts:HDSM283L
- added IC1: 74AHC138D,118, SamacSys_Parts:SOIC127P600X175-16N
- added IC3: ADP3339AKCZ-3.3-R7, SamacSys_Parts:SOT230P700X180-4N
- added IC4: SN74LVC1G19DBVRE4, SamacSys_Parts:SOT95P280X145-6N
- added J1: UJ2-MIBH-G-SMT-TR, SamacSys_Parts:UJ2MIBHGSMTTR
- added R2: 10k, adafruit:R0402
- added R3: 16, adafruit:R0402
- added S1, S2: KXT321LHS, SamacSys_Parts:KXT321LHS
- added S3: KMT221GHFLFS, SamacSys_Parts:KMT221GHFLFS
- C1, C2: device adafruit:C0805 -> adafruit:C0402
- C3: value .1uF -> 1uF; device adafruit:C0805 -> adafruit:C0402
- C4: value 2.2uF -> 1uF; device adafruit:C0805 -> adafruit:C0402
- R1: device adafruit:M0805 -> adafruit:R0402
- moved LED9 150.4 mm to (52.5, 129.5)
- moved U3 145.7 mm to (104.0, 19.3), turned to 270 degrees
- moved LED10 133.6 mm to (22.5, 129.5)
- moved LED7 133.6 mm to (65.2, 86.8)
- moved LED8 126.0 mm to (37.6, 114.4)
- moved LED15 120.4 mm to (9.90, 86.6)
- moved IC2 119.9 mm to (49.2, 8.02), turned to 270 degrees
- moved LED11 113.3 mm to (9.77, 108.6)
- moved LED5 113.2 mm to (59.4, 59.3)
- moved LED12 103.3 mm to (-5.45, 101.9)
- moved LED4 100.4 mm to (52.9, 43.9)
- moved LED13 98.4 mm to (-12.2, 86.7)
- moved LED6 98.3 mm to (37.5, 59.3)
- moved LED14 95.3 mm to (-5.26, 71.4)
- moved C2 94.3 mm to (48.8, 118.3), turned to 180 degrees
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Connections:
- removed net 3V3: U3.2
- new net CATH_A: IC1.15
- new net CATH_B: IC1.14
- new net CATH_C: IC1.13
- new net CATH_D: IC1.12
- new net CATH_DP1: IC1.7
- new net CATH_E: IC1.11
- new net CATH_F: IC1.10
- new net CATH_G: IC1.9
- new net COMM_ANODE: DS1.10, R3.2
- new net EN: C6.1, C7.1, R2.1, S2.2, U3.3
- new net GPIO0: C5.1, S1.2, U3.27
- new net GPIO12: S3.1, U3.20
- new net GPIO19: D2.1, J1.3, U3.13
- new net GPIO20: D1.1, J1.4, U3.14
- new net GPIO9: IC2.2, U3.17
- new net N$19: IC4.6, R3.1
- new net N$20: DS1.11
- new net N$21: DS1.1
- new net N$22: DS1.3
- new net N$23: DS1.4
- new net N$24: DS1.6
- net +3V3: now also C3.1, C8.1, IC1.16, IC1.6, IC3.2, IC3.4, IC4.5, R2.2, S3.3, U3.2; no longer C4.1, VOLTAGE_REG.5
- net +5V: now also C4.1, IC3.3, LED1.2, LED10.2, LED11.2, LED12.2, LED13.2, LED14.2, LED15.2, LED2.2, LED3.2, LED4.2, LED5.2, LED6.2, LED7.2, LED8.2, LED9.2; no longer C3.1, VOLTAGE_REG.1, VOLTAGE_REG.2
- net GND: now also C1.2, C2.2, C5.2, C6.2, C7.2, C8.2, D1.2, D2.2, IC1.4, IC1.5, IC1.8, IC3.1, IC4.2, IC4.3, J1.2, J1.MP1, J1.MP2, J1.MP3, J1.MP4, S1.1, S2.1, S3.5; no longer VOLTAGE_REG.3, VOLTAGE_REG.6
- net N$1: now also LED1.3, LED2.1; no longer LED1.1, LED2.3
- net N$15: now also LED1.1; no longer LED2.1
- net N$16: now also DS1.9; no longer C1.2, LED1.2, LED2.2, LED3.2, LED4.2, LED5.2, LED6.2, LED7.2, LED8.2
- net N$17: now also DS1.8; no longer C2.2, LED10.2, LED11.2, LED12.2, LED13.2, LED14.2, LED15.2, LED9.2
- net N$18: now also DS1.7; no longer IC2.2
- net N$2: now also LED2.3; no longer LED1.3
Routing:
- net +5V: track 0.00 -> 459.7 mm, vias 0 -> 4
- net +3V3: track 0.00 -> 223.1 mm, vias 0 -> 2
- net GPIO9: track 0.00 -> 48.2 mm, vias 0 -> 4
- net GPIO19: track 0.00 -> 40.6 mm
- net LED_CONTROL: track 0.00 -> 40.2 mm, vias 0 -> 2
- net N$7: track 0.00 -> 39.6 mm
- net GPIO20: track 0.00 -> 39.0 mm
- net N$6: track 0.00 -> 37.8 mm
- net EN: track 0.00 -> 35.0 mm, vias 0 -> 2
- net N$9: track 0.00 -> 32.4 mm
- net N$10: track 0.00 -> 29.6 mm
- net N$5: track 0.00 -> 24.3 mm
- net N$1: track 0.00 -> 21.7 mm
- net N$11: track 0.00 -> 21.5 mm
- net N$12: track 0.00 -> 21.5 mm
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- added copper zone on layer 1, net GND
- added copper zone on layer 16, net GND
Other:
- board size 247 x 191.8 mm -> 138 x 144.8 mm
- board text added: "Avant Gardens"
- board text added: "Boot"
- board text added: "Club Station Alpha"
- board text added: "Crux Prime"
- board text added: "Deep Freeze"
- board text added: "Forbidden Valley"
- board text added: "Gnarled Forest"
- board text added: "JLCJLCJLCJLC"
- board text added: "Moonbase"
- board text added: "Nexus Tower"
- board text added: "Nimbus Station"
- board text added: "Ninjago"
- board text added: "Pet Cove"
- board text added: "Portabello"
- board text added: "Reset"
- board text added: "Robot City"
- board text added: "Starbase 3001"
- board text added: "The Venture Explorer"
