File: LU Player Tracker Board V1/board.sch (EAGLE design)
At the start: 24 parts, among them IC2 TXU0304PWR, U3 ESP32-S3-WROOM-1-N16R2

Commit message: update
Parts:
- removed VOLTAGE_REG: TLS850B0TBV33ATMA1, SamacSys_Parts:TLS850B0TBV33ATMA1
- added C5, C6: .1uF, adafruit:C-USC0402
- added C7, C8: 1uF, adafruit:C-USC0402
- added D1, D2: ESD9L5.0ST5G, SamacSys_Parts:ESD9L5.0ST5G
- added DS1: HDSM-291C, SamacSys_Parts:HDSM-291C
- added IC1: 74AHC138D,118, SamacSys_Parts:74AHC138D,118
- added IC3: ADP3339AKCZ-3.3-R7, SamacSys_Parts:ADP3339AKCZ-3.3-R7
- added IC4: SN74LVC1G19DBVRE4, SamacSys_Parts:SN74LVC1G19DBVRE4
- added J1: UJ2-MIBH-G-SMT-TR, SamacSys_Parts:UJ2-MIBH-G-SMT-TR
- added R2: 10k, adafruit:R-US_R0402
- added R3: 16, adafruit:R-US_R0402
- added S1, S2: KXT321LHS, SamacSys_Parts:KXT321LHS
- added S3: KMT221GHFLFS, SamacSys_Parts:KMT221GHFLFS
- C1, C2: device adafruit:C-USC0805 -> adafruit:C-USC0402
- C3: value .1uF -> 1uF; device adafruit:C-USC0805 -> adafruit:C-USC0402
- C4: value 2.2uF -> 1uF; device adafruit:C-USC0805 -> adafruit:C-USC0402
- R1: device adafruit:R-US_M0805 -> adafruit:R-US_R0402
Connections:
- new net CATH_A: IC1.!Y0
- new net CATH_B: IC1.!Y1
- new net CATH_C: IC1.!Y2
- new net CATH_D: IC1.!Y3
- new net CATH_DP1: IC1.!Y7
- new net CATH_E: IC1.!Y4
- new net CATH_F: IC1.!Y5
- new net CATH_G: IC1.!Y6
- new net COMM_ANODE: DS1.COMMON_ANODE_DIG1, R3.2
- new net EN: C6.1, C7.1, R2.1, S2.NO, U3.EN
- new net GPIO0: C5.1, S1.NO, U3.IO0
- new net GPIO12: S3.NO_1, U3.IO12
- new net GPIO19: D2.K, J1.3, U3.IO19
- new net GPIO20: D1.K, J1.4, U3.IO20
- new net GPIO9: IC2.A1, U3.IO9
- new net N$19: IC4.Y0, R3.1
- new net N$20: DS1.CATHODE_DP1._DP3
- new net N$21: DS1.CATHODE_G
- new net N$22: DS1.CATHODE_A
- new net N$23: DS1.CATHODE_F
- new net N$24: DS1.CATHODE_D
- net +3V3: now also C3.1, C8.1, IC1.E3, IC1.VCC, IC3.OUT_1, IC3.OUT_2, IC4.VCC, R2.2, S3.COM_1, U3.3V3; no longer C4.1, VOLTAGE_REG.Q
- net +5V: now also C4.1, IC3.IN, LED1.VDD, LED10.VDD, LED11.VDD, LED12.VDD, LED13.VDD, LED14.VDD, LED15.VDD, LED2.VDD, LED3.VDD, LED4.VDD, LED5.VDD, LED6.VDD, LED7.VDD, LED8.VDD, LED9.VDD; no longer C3.1, VOLTAGE_REG.EN, VOLTAGE_REG.I
- net GND: now also C1.2, C2.2, C5.2, C6.2, C7.2, C8.2, D1.A, D2.A, IC1.!E1, IC1.!E2, IC1.GND, IC3.GND, IC4.!E, IC4.GND, J1.2, J1.MP1, J1.MP2, J1.MP3, J1.MP4, S1.COM, S2.COM, S3.GROUND, U3.GND; no longer VOLTAGE_REG.GND, VOLTAGE_REG.TAB
- net N$1: now also LED1.DOUT, LED2.DIN; no longer LED1.DIN, LED2.DOUT
- net N$15: now also LED1.DIN; no longer LED2.DIN
- net N$16: now also DS1.CATHODE_B; no longer C1.2, LED1.VDD, LED2.VDD, LED3.VDD, LED4.VDD, LED5.VDD, LED6.VDD, LED7.VDD, LED8.VDD
- net N$17: now also DS1.CATHODE_C; no longer C2.2, LED10.VDD, LED11.VDD, LED12.VDD, LED13.VDD, LED14.VDD, LED15.VDD, LED9.VDD
- net N$18: now also DS1.CATHODE_E; no longer IC2.A1
- net N$2: now also LED2.DOUT; no longer LED1.DOUT
Other:
- note added: "Boot"
- note added: "Mode"
- note added: "Reset"
