File: LU Player Tracker Board V2/board.brd (EAGLE design)
At the start: 138 x 144.8 mm, 39 parts, among them IC1 74AHC138D,118, IC2 TXU0304PWR, IC3 ADP3339AKCZ-3.3-R7, IC4 SN74LVC1G19DBVRE4, J1 UJ2-MIBH-G-SMT-TR, U3 ESP32-S3-WROOM-1-N16R2

Commit message: Updated to V2
Parts:
- added D3: ESD9L5.0ST5G, SamacSys_Parts:SODFL1006X40N
- added R4: 16, adafruit:R0402
- added R5: 0, adafruit:R0402
- C8: value 1uF -> .1uF
- DS1: device SamacSys_Parts:HDSM283L -> SamacSys_Parts:HDSM291C
Connections:
- net COMM_ANODE renamed COMM_ANODE_DIG1
- removed net N$17: DS1.8
- removed net N$18: DS1.7
- removed net N$20: DS1.11
- removed net N$21: DS1.1
- removed net N$22: DS1.3
- removed net N$23: DS1.4
- removed net N$24: DS1.6
- new net COMM_ANODE_DIG2: DS1.2, R4.2
- new net GPIO4: IC1.1, U3.4
- new net GPIO5: IC1.2, U3.5
- new net GPIO6: IC1.3, U3.6
- new net GPIO7: IC4.1, U3.7
- new net N$25: IC4.4, R4.1
- net +3V3: now also R5.2; no longer S3.3
- net +5V: now also D3.1
- net CATH_A: now also DS1.3
- net CATH_B: now also DS1.9
- net CATH_C: now also DS1.8
- net CATH_D: now also DS1.6
- net CATH_DP1: now also DS1.11
- net CATH_E: now also DS1.7
- net CATH_F: now also DS1.4
- net CATH_G: now also DS1.1
- net GND: now also D3.2
- net N$16: now also R5.1, S3.3; no longer DS1.9
Routing:
- net GPIO7: track 0.00 -> 95.0 mm, vias 0 -> 2
- net GPIO4: track 0.00 -> 90.1 mm, vias 0 -> 2
- net GPIO5: track 0.00 -> 90.0 mm, vias 0 -> 2
- net GPIO6: track 0.00 -> 89.8 mm, vias 0 -> 2
- net +3V3: track 223.1 -> 306.6 mm
- net CATH_G: track 0.00 -> 40.6 mm, vias 0 -> 2
- net CATH_DP1: track 0.00 -> 40.0 mm, vias 0 -> 2
- net CATH_C: track 0.00 -> 38.6 mm, vias 0 -> 2
- net CATH_B: track 0.00 -> 36.5 mm, vias 0 -> 2
- net CATH_E: track 0.00 -> 36.0 mm, vias 0 -> 2
- net CATH_D: track 0.00 -> 29.9 mm
- net CATH_F: track 0.00 -> 28.8 mm, vias 0 -> 2
- net CATH_A: track 0.00 -> 26.5 mm
- net COMM_ANODE_DIG1: track 0.00 -> 25.5 mm, vias 0 -> 2
- net COMM_ANODE_DIG2: track 0.00 -> 14.2 mm
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Other:
- board text added: "<- Aux World Occupied"
- board text added: "LU Player Tracker V2"
- board text added: "Ninjago Monastery"
- board text added: "Player Count"
- board text removed: "Ninjago"
