File: LU Player Tracker Board V2/board.sch (EAGLE design)
At the start: 39 parts, among them IC1 74AHC138D,118, IC2 TXU0304PWR, IC3 ADP3339AKCZ-3.3-R7, IC4 SN74LVC1G19DBVRE4, J1 UJ2-MIBH-G-SMT-TR, U3 ESP32-S3-WROOM-1-N16R2

Commit message: Updated to V2
Parts:
- added D3: ESD9L5.0ST5G, SamacSys_Parts:ESD9L5.0ST5G
- added R4: 16, adafruit:R-US_R0402
- added R5: 0, adafruit:R-US_R0402
- C8: value 1uF -> .1uF
Connections:
- net COMM_ANODE renamed COMM_ANODE_DIG1
- removed net N$17: DS1.CATHODE_C
- removed net N$18: DS1.CATHODE_E
- removed net N$20: DS1.CATHODE_DP1._DP3
- removed net N$21: DS1.CATHODE_G
- removed net N$22: DS1.CATHODE_A
- removed net N$23: DS1.CATHODE_F
- removed net N$24: DS1.CATHODE_D
- new net COMM_ANODE_DIG2: DS1.CATHODE_DP2._DP4, R4.2
- new net GPIO4: IC1.A0, U3.IO4
- new net GPIO5: IC1.A1, U3.IO5
- new net GPIO6: IC1.A2, U3.IO6
- new net GPIO7: IC4.A, U3.IO7
- new net N$25: IC4.Y1, R4.1
- net +3V3: now also R5.2; no longer S3.COM_1
- net +5V: now also D3.K
- net CATH_A: now also DS1.CATHODE_A
- net CATH_B: now also DS1.CATHODE_B
- net CATH_C: now also DS1.CATHODE_C
- net CATH_D: now also DS1.CATHODE_D
- net CATH_DP1: now also DS1.CATHODE_DP1._DP3
- net CATH_E: now also DS1.CATHODE_E
- net CATH_F: now also DS1.CATHODE_F
- net CATH_G: now also DS1.CATHODE_G
- net GND: now also D3.A
- net N$16: now also R5.1, S3.COM_1; no longer DS1.CATHODE_B
Other:
- note added: "Boot Btn"
- note added: "Mode Btn"
- note added: "Reset Btn"
- note removed: "Boot"
- note removed: "Mode"
- note removed: "Reset"
- moved on the sheet: DS1, R3
