File: LU Player Tracker Board V3/board.brd (EAGLE design)
At the start: 138 x 144.8 mm, 42 parts, among them IC1 74AHC138D,118, IC2 TXU0304PWR, IC3 ADP3339AKCZ-3.3-R7, IC4 SN74LVC1G19DBVRE4, J1 UJ2-MIBH-G-SMT-TR, U3 ESP32-S3-WROOM-1-N16R2

Commit message: v3 of board
Parts:
- removed R5: 0, adafruit:R0402
Connections:
- removed net CATH_DP1: DS1.11, IC1.7
- removed net N$16: R5.1, S3.3
- new net CATH_DP2: DS1.2, IC1.7
- net +3V3: now also DS1.11, S3.3; no longer R5.2
- net COMM_ANODE_DIG2: now also DS1.5; no longer DS1.2
Routing:
- net CATH_DP1: track 40.0 -> 0.00 mm, vias 2 -> 0
- net CATH_DP2: track 0.00 -> 38.5 mm, vias 0 -> 2
- net +3V3: track 306.6 -> 344.1 mm, vias 2 -> 4
- net N$16: track 5.71 -> 0.00 mm
- net COMM_ANODE_DIG2: track 14.2 -> 17.0 mm, vias 0 -> 2
- net CATH_F: track 28.8 -> 28.0 mm
Other:
- board text added: "LU Player Tracker V3"
- board text removed: "LU Player Tracker V2"
Changed lines of the file:
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@@
 <drawing>
 <settings>
-<setting alwaysvectorfont="yes"/>
+<setting alwaysvectorfont="no"/>
 <setting verticaltext="up"/>
 </settings>
@@
     Occupied</text>
 <text x="82.944" y="137.719" size="1.4224" layer="21">Player Count</text>
-<text x="-23" y="141" size="1.778" layer="21">LU Player Tracker V2</text>
+<text x="-23" y="141" size="1.778" layer="21">LU Player Tracker V3</text>
 </plain>
 <attributes>
@@
 <attribute name="MOUSER_PRICE-STOCK" value="https://www.mouser.co.uk/ProductDetail/onsemi/ESD9L5.0ST5G?qs=lq5%252BOP7PS0%252BtbEEODUxZiA%3D%3D" x="-12.526" y="15.64" size="1.778" layer="27" rot="R90" display="off"/>
 </element>
-<element name="R5" library="adafruit" library_urn="urn:adsk.eagle:library:420" package="R0402" package3d_urn="urn:adsk.eagle:package:6240564/1" override_package3d_urn="urn:adsk.eagle:package:38544695/3" override_package_urn="urn:adsk.eagle:footprint:6239918/1" value="0" x="88.964" y="5.283" smashed="yes" rot="R270">
-<attribute name="NAME" x="89.726" y="5.918" size="0.6096" layer="25" rot="R270"/>
-</element>
 </elements>
 <signals>
@@
 <wire x1="85" y1="103" x2="84" y2="104" width="0.1524" layer="1"/>
 <wire x1="92" y1="47" x2="90" y2="45" width="0.1524" layer="1"/>
-<contactref element="R5" pad="2"/>
 <wire x1="88" y1="2.3942" x2="88.3942" y2="2.3942" width="0.1524" layer="1"/>
 <wire x1="88.3942" y1="2.3942" x2="89" y2="3" width="0.1524" layer="1"/>
 <wire x1="89" y1="3" x2="89" y2="4.597" width="0.1524" layer="1"/>
-<wire x1="89" y1="4.597" x2="88.964" y2="4.633" width="0.1524" layer="1"/>
+<contactref element="DS1" pad="11"/>
+<wire x1="81.25" y1="104" x2="80.15" y2="104" width="0.1524" layer="1"/>
+<wire x1="80" y1="104.15" x2="80" y2="119" width="0.1524" layer="1"/>
+<via x="80" y="119" extent="1-16" drill="0.35"/>
+<wire x1="80" y1="119" x2="80" y2="126.609" width="0.1524" layer="16"/>
+<wire x1="80" y1="126.609" x2="83.947" y2="130.556" width="0.1524" layer="16"/>
+<via x="83.947" y="130.556" extent="1-16" drill="0.35"/>
+<wire x1="83.947" y1="130.556" x2="83.947" y2="133.007" width="0.1524" layer="1"/>
+<wire x1="83.947" y1="133.007" x2="84.19" y2="133.25" width="0.1524" layer="1"/>
+<wire x1="80.15" y1="104" x2="80" y2="104.15" width="0.1524" layer="1"/>
+<contactref element="S3" pad="3"/>
+<wire x1="92.456" y1="4.953" x2="93.466" y2="3.943" width="0.1524" layer="1"/>
+<wire x1="93.466" y1="3.943" x2="93.466" y2="3.558" width="0.1524" layer="1"/>
+<wire x1="89" y1="4.597" x2="89.356" y2="4.953" width="0.1524" layer="1"/>
+<wire x1="89.356" y1="4.953" x2="92.456" y2="4.953" width="0.1524" layer="1"/>
 </signal>
 <signal name="N$2">
@@
 <via x="98.425" y="99.822" extent="1-16" drill="0.35"/>
 <wire x1="98.425" y1="99.822" x2="93.472" y2="104.775" width="0.1524" layer="16"/>
-<wire x1="91" y1="116" x2="91" y2="120" width="0.1524" layer="16"/>
-<via x="91" y="120" extent="1-16" drill="0.35"/>
+<wire x1="89.603" y1="117.397" x2="89.603" y2="119.873" width="0.1524" layer="16"/>
+<via x="89.603" y="119.873" extent="1-16" drill="0.35"/>
 <wire x1="93.472" y1="104.775" x2="93.472" y2="113.528" width="0.1524" layer="16"/>
-<wire x1="93.472" y1="113.528" x2="91" y2="116" width="0.1524" layer="16"/>
-<wire x1="91" y1="120" x2="89.677" y2="120" width="0.1524" layer="1"/>
+<wire x1="93.472" y1="113.528" x2="89.603" y2="117.397" width="0.1524" layer="16"/>
+<wire x1="89.603" y1="119.873" x2="89.603" y2="120.074" width="0.1524" layer="1"/>
 <wire x1="89.27" y1="120.407" x2="89.27" y2="122.75" width="0.1524" layer="1"/>
-<wire x1="89.677" y1="120" x2="89.27" y2="120.407" width="0.1524" layer="1"/>
+<wire x1="89.603" y1="120.074" x2="89.27" y2="120.407" width="0.1524" layer="1"/>
 </signal>
 <signal name="CATH_G">
@@
 <wire x1="86.487" y1="103.513" x2="86.487" y2="117.513" width="0.1524" layer="16"/>
 </signal>
-<signal name="CATH_DP1">
-<contactref element="IC1" pad="7"/>
-<contactref element="DS1" pad="11"/>
-<via x="96.901" y="102.489" extent="1-16" drill="0.35"/>
-<wire x1="94.275" y1="99.825" x2="94.9664" y2="100.5164" width="0.1524" layer="1"/>
-<wire x1="94.9664" y1="100.5164" x2="95.1446875" y2="100.5164" width="0.1524" layer="1"/>
-<wire x1="95.1446875" y1="100.5164" x2="96.901" y2="102.2727125" width="0.1524" layer="1"/>
-<wire x1="96.901" y1="102.2727125" x2="96.901" y2="102.489" width="0.1524" layer="1"/>
-<wire x1="96.901" y1="102.489" x2="96.901" y2="113.284" width="0.1524" layer="16"/>
-<wire x1="92" y1="118.185" x2="92" y2="122" width="0.1524" layer="16"/>
-<wire x1="92" y1="122" x2="87" y2="127" width="0.1524" layer="16"/>
-<via x="87" y="127" extent="1-16" drill="0.35"/>
-<wire x1="96.901" y1="113.284" x2="92" y2="118.185" width="0.1524" layer="16"/>
-<wire x1="87" y1="127" x2="84" y2="130" width="0.1524" layer="1"/>
-<wire x1="84" y1="130" x2="84" y2="133.06" width="0.1524" layer="1"/>
-<wire x1="84" y1="133.06" x2="84.19" y2="133.25" width="0.1524" layer="1"/>
-</signal>
 <signal name="N$19">
 <contactref element="IC4" pad="6"/>
@@
 <signal name="COMM_ANODE_DIG2">
 <contactref element="R4" pad="2"/>
-<contactref element="DS1" pad="2"/>
-<wire x1="87.65" y1="110" x2="87.65" y2="118.217" width="0.1524" layer="1"/>
-<wire x1="84.19" y1="121.677" x2="84.19" y2="122.75" width="0.1524" layer="1"/>
-<wire x1="87.65" y1="118.217" x2="84.19" y2="121.677" width="0.1524" layer="1"/>
+<contactref element="DS1" pad="5"/>
+<wire x1="87.65" y1="110" x2="87.759" y2="110.109" width="0.1524" layer="1"/>
+<wire x1="87.759" y1="110.109" x2="90.932" y2="110.109" width="0.1524" layer="1"/>
+<wire x1="90.932" y1="110.109" x2="91.44" y2="110.617" width="0.1524" layer="1"/>
+<wire x1="91.44" y1="116.84" x2="91.567" y2="116.967" width="0.1524" layer="1"/>
+<via x="91.567" y="116.967" extent="1-16" drill="0.35"/>
+<wire x1="91.567" y1="116.967" x2="91" y2="117.534" width="0.1524" layer="16"/>
+<wire x1="91" y1="117.534" x2="91" y2="119" width="0.1524" layer="16"/>
+<via x="91" y="119" extent="1-16" drill="0.35"/>
+<wire x1="91" y1="119" x2="92" y2="120" width="0.1524" layer="1"/>
+<wire x1="92" y1="120" x2="92" y2="122.56" width="0.1524" layer="1"/>
+<wire x1="92" y1="122.56" x2="91.81" y2="122.75" width="0.1524" layer="1"/>
+<wire x1="91.44" y1="110.617" x2="91.44" y2="116.84" width="0.1524" layer="1"/>
 </signal>
 <signal name="GPIO4">
@@
 <wire x1="78.7" y1="105" x2="78.75" y2="104.95" width="0.1524" layer="1"/>
 </signal>
-<signal name="N$16">
-<contactref element="R5" pad="1"/>
-<contactref element="S3" pad="3"/>
-<wire x1="88.964" y1="5.933" x2="90.067" y2="5.933" width="0.1524" layer="1"/>
-<wire x1="91.047" y1="4.953" x2="92.456" y2="4.953" width="0.1524" layer="1"/>
-<wire x1="92.456" y1="4.953" x2="93.466" y2="3.943" width="0.1524" layer="1"/>
-<wire x1="93.466" y1="3.943" x2="93.466" y2="3.558" width="0.1524" layer="1"/>
-<wire x1="90.067" y1="5.933" x2="91.047" y2="4.953" width="0.1524" layer="1"/>
+<signal name="CATH_DP2">
+<contactref element="DS1" pad="2"/>
+<contactref element="IC1" pad="7"/>
+<via x="96.901" y="102.489" extent="1-16" drill="0.35"/>
+<wire x1="94.275" y1="99.825" x2="94.9664" y2="100.5164" width="0.1524" layer="1"/>
+<wire x1="94.9664" y1="100.5164" x2="95.1446875" y2="100.5164" width="0.1524" layer="1"/>
+<wire x1="95.1446875" y1="100.5164" x2="96.901" y2="102.2727125" width="0.1524" layer="1"/>
+<wire x1="96.901" y1="102.2727125" x2="96.901" y2="102.489" width="0.1524" layer="1"/>
+<wire x1="96.901" y1="102.489" x2="96.901" y2="113.284" width="0.1524" layer="16"/>
+<wire x1="92" y1="118.185" x2="92" y2="122" width="0.1524" layer="16"/>
+<wire x1="92" y1="122" x2="87" y2="127" width="0.1524" layer="16"/>
+<via x="87" y="127" extent="1-16" drill="0.35"/>
+<wire x1="96.901" y1="113.284" x2="92" y2="118.185" width="0.1524" layer="16"/>
+<wire x1="87" y1="127" x2="86" y2="127" width="0.1524" layer="1"/>
+<wire x1="86" y1="127" x2="84.19" y2="125.19" width="0.1524" layer="1"/>
+<wire x1="84.19" y1="125.19" x2="84.19" y2="122.75" width="0.1524" layer="1"/>
 </signal>
 </signals>

Commit message: resistor change
Parts:
- R3, R4: value 16 -> 100
Changed lines of the file:
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@@
 <attribute name="NAME" x="80" y="104.079" size="0.6096" layer="25" align="center"/>
 </element>
-<element name="R3" library="adafruit" library_urn="urn:adsk.eagle:library:420" package="R0402" package3d_urn="urn:adsk.eagle:package:6240564/1" override_package3d_urn="urn:adsk.eagle:package:38544695/2" override_package_urn="urn:adsk.eagle:footprint:6239918/1" value="16" x="83" y="110" smashed="yes">
+<element name="R3" library="adafruit" library_urn="urn:adsk.eagle:library:420" package="R0402" package3d_urn="urn:adsk.eagle:package:6240564/1" override_package3d_urn="urn:adsk.eagle:package:38544695/2" override_package_urn="urn:adsk.eagle:footprint:6239918/1" value="100" x="83" y="110" smashed="yes">
 <attribute name="NAME" x="82.365" y="110.762" size="0.6096" layer="25"/>
 <attribute name="VALUE" x="82.619" y="108.73" size="0.6096" layer="27"/>
@@
 <attribute name="NAME" x="90.54" y="128.006" size="0.6096" layer="25" align="center"/>
 </element>
-<element name="R4" library="adafruit" library_urn="urn:adsk.eagle:library:420" package="R0402" package3d_urn="urn:adsk.eagle:package:6240564/1" override_package3d_urn="urn:adsk.eagle:package:38544695/2" override_package_urn="urn:adsk.eagle:footprint:6239918/1" value="16" x="87" y="110" smashed="yes">
+<element name="R4" library="adafruit" library_urn="urn:adsk.eagle:library:420" package="R0402" package3d_urn="urn:adsk.eagle:package:6240564/1" override_package3d_urn="urn:adsk.eagle:package:38544695/2" override_package_urn="urn:adsk.eagle:footprint:6239918/1" value="100" x="87" y="110" smashed="yes">
 <attribute name="NAME" x="86.365" y="110.762" size="0.6096" layer="25"/>
 <attribute name="VALUE" x="86.619" y="108.73" size="0.6096" layer="27"/>
