File: LU Player Tracker Board V3/board.sch (EAGLE design)
At the start: 42 parts, among them IC1 74AHC138D,118, IC2 TXU0304PWR, IC3 ADP3339AKCZ-3.3-R7, IC4 SN74LVC1G19DBVRE4, J1 UJ2-MIBH-G-SMT-TR, U3 ESP32-S3-WROOM-1-N16R2

Commit message: v3 of board
Parts:
- removed R5: 0, adafruit:R-US_R0402
Connections:
- removed net CATH_DP1: DS1.CATHODE_DP1._DP3, IC1.!Y7
- removed net N$16: R5.1, S3.COM_1
- new net CATH_DP2: DS1.CATHODE_DP2._DP4, IC1.!Y7
- net +3V3: now also DS1.CATHODE_DP1._DP3, S3.COM_1; no longer R5.2
- net COMM_ANODE_DIG2: now also DS1.COMMON_ANODE_DIG2; no longer DS1.CATHODE_DP2._DP4
Other:
- note added: "LOW = dig 2 HIGH = dig 1 dig 1 | dig 2"
Changed lines of the file:
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@@
 <part name="D3" library="SamacSys_Parts" deviceset="ESD9L5.0ST5G" device="" override_package3d_urn="urn:adsk.eagle:package:38544704/2" override_package_urn="urn:adsk.eagle:footprint:38544705/1"/>
 <part name="SUPPLY31" library="supply2" library_urn="urn:adsk.eagle:library:372" deviceset="GND" device=""/>
-<part name="R5" library="adafruit" library_urn="urn:adsk.eagle:library:420" deviceset="R-US_" device="R0402" package3d_urn="urn:adsk.eagle:package:6240564/1" override_package3d_urn="urn:adsk.eagle:package:38544695/3" override_package_urn="urn:adsk.eagle:footprint:6239918/1" value="0"/>
+<part name="+3V6" library="supply1" library_urn="urn:adsk.eagle:library:371" deviceset="+3V3" device=""/>
 </parts>
 <sheets>
@@
 <attribute name="VALUE" x="254.635" y="154.305" size="1.778" layer="96"/>
 </instance>
-<instance part="R5" gate="G$1" x="83.82" y="162.56" smashed="yes" rot="R180">
-<attribute name="NAME" x="87.63" y="161.0614" size="1.778" layer="95" rot="R180"/>
-<attribute name="VALUE" x="87.63" y="165.862" size="1.778" layer="96" rot="R180"/>
-</instance>
 </instances>
 <busses>
@@
 <wire x1="71.12" y1="162.56" x2="71.12" y2="170.18" width="0.1524" layer="91"/>
 <pinref part="+3V5" gate="G$1" pin="+3V3"/>
-<pinref part="R5" gate="G$1" pin="2"/>
-<wire x1="71.12" y1="162.56" x2="78.74" y2="162.56" width="0.1524" layer="91"/>
+<pinref part="S3" gate="G$1" pin="COM_1"/>
+<wire x1="71.12" y1="162.56" x2="96.52" y2="162.56" width="0.1524" layer="91"/>
 </segment>
 <segment>
@@
 <wire x1="205.74" y1="119.38" x2="195.58" y2="119.38" width="0.1524" layer="91"/>
 <label x="195.58" y="119.38" size="1.778" layer="95"/>
-</segment>
-</net>
-<net name="N$16" class="0">
-<segment>
-<pinref part="R5" gate="G$1" pin="1"/>
-<pinref part="S3" gate="G$1" pin="COM_1"/>
-<wire x1="88.9" y1="162.56" x2="96.52" y2="162.56" width="0.1524" layer="91"/>
 </segment>
 </net>
@@
 <description>7-segment</description>
 <plain>
+<text x="208.28" y="104.14" size="1.778" layer="91">LOW = dig 2
+HIGH = dig 1
+dig 1 |  dig 2</text>
 </plain>
 <instances>
@@
 <attribute name="VALUE" x="267.97" y="88.138" size="1.778" layer="96"/>
 </instance>
+<instance part="+3V6" gate="G$1" x="228.6" y="215.9" smashed="yes">
+<attribute name="VALUE" x="231.14" y="218.44" size="1.778" layer="96" rot="R180"/>
+</instance>
 </instances>
 <busses>
@@
 <wire x1="116.84" y1="101.6" x2="116.84" y2="104.14" width="0.1524" layer="91"/>
 <pinref part="+3V8" gate="G$1" pin="+3V3"/>
+</segment>
+<segment>
+<pinref part="DS1" gate="G$1" pin="CATHODE_DP1._DP3"/>
+<wire x1="224.282" y1="205.74" x2="228.6" y2="205.74" width="0.1524" layer="91"/>
+<wire x1="228.6" y1="205.74" x2="228.6" y2="213.36" width="0.1524" layer="91"/>
+<pinref part="+3V6" gate="G$1" pin="+3V3"/>
 </segment>
 </net>
@@
 </segment>
 </net>
-<net name="CATH_DP1" class="0">
+<net name="N$19" class="0">
+<segment>
+<pinref part="IC4" gate="G$1" pin="Y0"/>
+<pinref part="R3" gate="G$1" pin="1"/>
+<wire x1="254" y1="99.06" x2="269.24" y2="99.06" width="0.1524" layer="91"/>
+</segment>
+</net>
+<net name="COMM_ANODE_DIG1" class="0">
+<segment>
+<wire x1="224.282" y1="203.2" x2="236.982" y2="203.2" width="0.1524" layer="91"/>
+<label x="236.982" y="203.2" size="1.778" layer="95" xref="yes"/>
+<pinref part="DS1" gate="G$1" pin="COMMON_ANODE_DIG1"/>
+</segment>
+<segment>
+<pinref part="R3" gate="G$1" pin="2"/>
+<wire x1="279.4" y1="99.06" x2="287.02" y2="99.06" width="0.1524" layer="91"/>
+<label x="287.02" y="99.06" size="1.778" layer="95" xref="yes"/>
+</segment>
+</net>
+<net name="N$25" class="0">
+<segment>
+<pinref part="IC4" gate="G$1" pin="Y1"/>
+<wire x1="254" y1="93.98" x2="266.7" y2="93.98" width="0.1524" layer="91"/>
+<wire x1="266.7" y1="93.98" x2="266.7" y2="91.44" width="0.1524" layer="91"/>
+<pinref part="R4" gate="G$1" pin="1"/>
+</segment>
+</net>
+<net name="COMM_ANODE_DIG2" class="0">
+<segment>
+<pinref part="R4" gate="G$1" pin="2"/>
+<wire x1="276.86" y1="91.44" x2="287.02" y2="91.44" width="0.1524" layer="91"/>
+<label x="287.02" y="91.44" size="1.778" layer="95" xref="yes"/>
+</segment>
+<segment>
+<pinref part="DS1" gate="G$1" pin="COMMON_ANODE_DIG2"/>
+<wire x1="163.322" y1="195.58" x2="152.4" y2="195.58" width="0.1524" layer="91"/>
+<label x="152.4" y="195.58" size="1.778" layer="95" rot="R180" xref="yes"/>
+</segment>
+</net>
+<net name="GPIO4" class="0">
+<segment>
+<pinref part="IC1" gate="G$1" pin="A0"/>
+<wire x1="127" y1="114.3" x2="119.38" y2="114.3" width="0.1524" layer="91"/>
+<label x="119.38" y="114.3" size="1.778" layer="95"/>
+</segment>
+</net>
+<net name="GPIO5" class="0">
+<segment>
+<pinref part="IC1" gate="G$1" pin="A1"/>
+<wire x1="127" y1="111.76" x2="119.38" y2="111.76" width="0.1524" layer="91"/>
+<label x="119.38" y="111.76" size="1.778" layer="95"/>
+</segment>
+</net>
+<net name="GPIO6" class="0">
+<segment>
+<pinref part="IC1" gate="G$1" pin="A2"/>
+<wire x1="127" y1="109.22" x2="119.38" y2="109.22" width="0.1524" layer="91"/>
+<label x="119.38" y="109.22" size="1.778" layer="95"/>
+</segment>
+</net>
+<net name="GPIO7" class="0">
+<segment>
+<pinref part="IC4" gate="G$1" pin="A"/>
+<wire x1="228.6" y1="99.06" x2="218.44" y2="99.06" width="0.1524" layer="91"/>
+<label x="218.44" y="99.06" size="1.778" layer="95"/>
+</segment>
+</net>
+<net name="CATH_DP2" class="0">
+<segment>
+<pinref part="DS1" gate="G$1" pin="CATHODE_DP2._DP4"/>
+<wire x1="163.322" y1="203.2" x2="152.4" y2="203.2" width="0.1524" layer="91"/>
+<label x="152.4" y="203.2" size="1.778" layer="95"/>
+</segment>
 <segment>
 <pinref part="IC1" gate="G$1" pin="!Y7"/>
@@
 <wire x1="124.46" y1="91.44" x2="142.24" y2="91.44" width="0.1524" layer="91"/>
 <label x="142.24" y="91.44" size="1.778" layer="95" xref="yes"/>
-</segment>
-<segment>
-<wire x1="224.282" y1="205.74" x2="236.982" y2="205.74" width="0.1524" layer="91"/>
-<pinref part="DS1" gate="G$1" pin="CATHODE_DP1._DP3"/>
-<label x="226.822" y="205.74" size="1.778" layer="95"/>
-</segment>
-</net>
-<net name="N$19" class="0">
-<segment>
-<pinref part="IC4" gate="G$1" pin="Y0"/>
-<pinref part="R3" gate="G$1" pin="1"/>
-<wire x1="254" y1="99.06" x2="269.24" y2="99.06" width="0.1524" layer="91"/>
-</segment>
-</net>
-<net name="COMM_ANODE_DIG1" class="0">
-<segment>
-<wire x1="224.282" y1="203.2" x2="236.982" y2="203.2" width="0.1524" layer="91"/>
-<label x="236.982" y="203.2" size="1.778" layer="95" xref="yes"/>
-<pinref part="DS1" gate="G$1" pin="COMMON_ANODE_DIG1"/>
-</segment>
-<segment>
-<pinref part="R3" gate="G$1" pin="2"/>
-<wire x1="279.4" y1="99.06" x2="287.02" y2="99.06" width="0.1524" layer="91"/>
-<label x="287.02" y="99.06" size="1.778" layer="95" xref="yes"/>
-</segment>
-</net>
-<net name="N$25" class="0">
-<segment>
-<pinref part="IC4" gate="G$1" pin="Y1"/>
-<wire x1="254" y1="93.98" x2="266.7" y2="93.98" width="0.1524" layer="91"/>
-<wire x1="266.7" y1="93.98" x2="266.7" y2="91.44" width="0.1524" layer="91"/>
-<pinref part="R4" gate="G$1" pin="1"/>
-</segment>
-</net>
-<net name="COMM_ANODE_DIG2" class="0">
-<segment>
-<pinref part="R4" gate="G$1" pin="2"/>
-<wire x1="276.86" y1="91.44" x2="287.02" y2="91.44" width="0.1524" layer="91"/>
-<label x="287.02" y="91.44" size="1.778" layer="95" xref="yes"/>
-</segment>
-<segment>
-<pinref part="DS1" gate="G$1" pin="CATHODE_DP2._DP4"/>
-<wire x1="163.322" y1="203.2" x2="153.162" y2="203.2" width="0.1524" layer="91"/>
-<label x="153.162" y="203.2" size="1.778" layer="95" rot="R180" xref="yes"/>
-</segment>
-</net>
-<net name="GPIO4" class="0">
-<segment>
-<pinref part="IC1" gate="G$1" pin="A0"/>
-<wire x1="127" y1="114.3" x2="119.38" y2="114.3" width="0.1524" layer="91"/>
-<label x="119.38" y="114.3" size="1.778" layer="95"/>
-</segment>
-</net>
-<net name="GPIO5" class="0">
-<segment>
-<pinref part="IC1" gate="G$1" pin="A1"/>
-<wire x1="127" y1="111.76" x2="119.38" y2="111.76" width="0.1524" layer="91"/>
-<label x="119.38" y="111.76" size="1.778" layer="95"/>
-</segment>
-</net>
-<net name="GPIO6" class="0">
-<segment>
-<pinref part="IC1" gate="G$1" pin="A2"/>
-<wire x1="127" y1="109.22" x2="119.38" y2="109.22" width="0.1524" layer="91"/>
-<label x="119.38" y="109.22" size="1.778" layer="95"/>
-</segment>
-</net>
-<net name="GPIO7" class="0">
-<segment>
-<pinref part="IC4" gate="G$1" pin="A"/>
-<wire x1="228.6" y1="99.06" x2="218.44" y2="99.06" width="0.1524" layer="91"/>
-<label x="218.44" y="99.06" size="1.778" layer="95"/>
 </segment>
 </net>
@@
 </drawing>
 <compatibility>
+<note version="6.3" minversion="6.2.2" severity="warning">
+Since Version 6.2.2 text objects can contain more than one line,
+which will not be processed correctly with this version.
+</note>
 <note version="8.2" severity="warning">
 Since Version 8.2, EAGLE supports online libraries. The ids

Commit message: resistor change
Parts:
- R3, R4: value 16 -> 100
Changed lines of the file:
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@@
 <part name="IC4" library="SamacSys_Parts" deviceset="SN74LVC1G19DBVRE4" device="" override_package3d_urn="urn:adsk.eagle:package:38561177/2" override_package_urn="urn:adsk.eagle:footprint:38561178/1"/>
 <part name="SUPPLY29" library="supply2" library_urn="urn:adsk.eagle:library:372" deviceset="GND" device=""/>
-<part name="R3" library="adafruit" library_urn="urn:adsk.eagle:library:420" deviceset="R-US_" device="R0402" package3d_urn="urn:adsk.eagle:package:6240564/1" override_package3d_urn="urn:adsk.eagle:package:38544695/2" override_package_urn="urn:adsk.eagle:footprint:6239918/1" value="16"/>
+<part name="R3" library="adafruit" library_urn="urn:adsk.eagle:library:420" deviceset="R-US_" device="R0402" package3d_urn="urn:adsk.eagle:package:6240564/1" override_package3d_urn="urn:adsk.eagle:package:38544695/2" override_package_urn="urn:adsk.eagle:footprint:6239918/1" value="100"/>
 <part name="+3V7" library="supply1" library_urn="urn:adsk.eagle:library:371" deviceset="+3V3" device=""/>
 <part name="SUPPLY30" library="supply2" library_urn="urn:adsk.eagle:library:372" deviceset="GND" device=""/>
@@
 <part name="+3V9" library="supply1" library_urn="urn:adsk.eagle:library:371" deviceset="+3V3" device=""/>
 <part name="DS1" library="SamacSys_Parts" deviceset="HDSM-291C" device="" override_package3d_urn="urn:adsk.eagle:package:38561171/2" override_package_urn="urn:adsk.eagle:footprint:38561172/1" override_locally_modified="yes"/>
-<part name="R4" library="adafruit" library_urn="urn:adsk.eagle:library:420" deviceset="R-US_" device="R0402" package3d_urn="urn:adsk.eagle:package:6240564/1" override_package3d_urn="urn:adsk.eagle:package:38544695/2" override_package_urn="urn:adsk.eagle:footprint:6239918/1" value="16"/>
+<part name="R4" library="adafruit" library_urn="urn:adsk.eagle:library:420" deviceset="R-US_" device="R0402" package3d_urn="urn:adsk.eagle:package:6240564/1" override_package3d_urn="urn:adsk.eagle:package:38544695/2" override_package_urn="urn:adsk.eagle:footprint:6239918/1" value="100"/>
 <part name="D3" library="SamacSys_Parts" deviceset="ESD9L5.0ST5G" device="" override_package3d_urn="urn:adsk.eagle:package:38544704/2" override_package_urn="urn:adsk.eagle:footprint:38544705/1"/>
 <part name="SUPPLY31" library="supply2" library_urn="urn:adsk.eagle:library:372" deviceset="GND" device=""/>
